File: Hardware/SmartSensor.sch (KiCad schematic (older format))
At the start: 4 parts

Commit message: Added final version 1.2 to the repository
Changed lines of the file:
@@
 Sheet 1 6
 Title "SmartSensor"
-Date "2021-03-19"
-Rev "1.1"
+Date "2021-06-14"
+Rev "1.2"
 Comp "Avans Hogeschool"
 Comment1 "Maurice Snoeren"
@@
 $EndSheet
 $Sheet
-S 1000 2250 1400 1100
-U 5F86FCBB
-F0 "Sensors" 50
-F1 "SmartSensor_Sensors.sch" 50
-F2 "CO2_ENABLE" I R 2400 2500 50
-F3 "LS_ENABLE" I R 2400 2600 50
-F4 "HT_ENABLE" I R 2400 2700 50
-F5 "SDA" B R 2400 2900 50
-F6 "SCL" I R 2400 3000 50
-F7 "RESET" I R 2400 2350 50
-F8 "CO2_INT" O R 2400 3150 50
-F9 "CO2_WAKE" O R 2400 3250 50
-$EndSheet
-$Sheet
 S 2900 1550 1400 3600
 U 5F76931A
@@
 F2 "ADAPTER_IN_USE" I L 2900 1850 50
 F3 "RESET" O L 2900 2350 50
-F4 "CO2_ENABLE" O L 2900 2500 50
-F5 "LS_ENABLE" O L 2900 2600 50
-F6 "THS_ENABLE" O L 2900 2700 50
-F7 "SDA" B L 2900 2900 50
-F8 "SCL" O L 2900 3000 50
-F9 "CO2_INT" O L 2900 3150 50
-F10 "CO2_WAKE" O L 2900 3250 50
-F11 "ATM_MOSI" O L 2900 4150 50
-F12 "ATM_MISO" I L 2900 4250 50
-F13 "ATM_CLK" O L 2900 4350 50
-F14 "ATM_TXD_0" O R 4300 3650 50
-F15 "ATM_TXD_1" O L 2900 3750 50
-F16 "ATM_RXD_0" I R 4300 3750 50
-F17 "ATM_RXD_1" I L 2900 3650 50
-F18 "XBEE_SS" O L 2900 4450 50
-F19 "XBEE_SLEEP" O L 2900 4650 50
-F20 "XBEE_ENABLE" O L 2900 4850 50
-F21 "RF_IRQ" I L 2900 5050 50
-F22 "ATM_PA0" T R 4300 4050 50
-F23 "ATM_PA1" T R 4300 4150 50
-F24 "ATM_PA2" T R 4300 4250 50
-F25 "ATM_MISO_1_RXD_2" I R 4300 4600 50
-F26 "ATM_MOSI_1_TXD_2" O R 4300 4500 50
-F27 "ATM_SCK_1" O R 4300 4700 50
-F28 "ATM_SDA_1" B R 4300 3250 50
-F29 "ATM_SCL_1" O R 4300 3350 50
-F30 "ATM_PA3" T R 4300 4350 50
-F31 "ATM_PB3" O R 4300 3850 50
-F32 "ATM_PB4" O R 4300 3950 50
+F4 "SDA" B L 2900 2900 50
+F5 "SCL" O L 2900 3000 50
+F6 "CO2_INT" O L 2900 3150 50
+F7 "CO2_WAKE" O L 2900 3250 50
+F8 "ATM_MOSI" O L 2900 4150 50
+F9 "ATM_MISO" I L 2900 4250 50
+F10 "ATM_CLK" O L 2900 4350 50
+F11 "ATM_TXD_0" O R 4300 3650 50
+F12 "ATM_TXD_1" O L 2900 3750 50
+F13 "ATM_RXD_0" I R 4300 3750 50
+F14 "ATM_RXD_1" I L 2900 3650 50
+F15 "XBEE_SS" O L 2900 4450 50
+F16 "XBEE_SLEEP" O L 2900 4650 50
+F17 "RF_IRQ" I L 2900 5050 50
+F18 "ATM_PA0" T R 4300 4050 50
+F19 "ATM_PA1" T R 4300 4150 50
+F20 "ATM_PA2" T R 4300 4250 50
+F21 "ATM_MISO_1_RXD_2" I R 4300 4600 50
+F22 "ATM_MOSI_1_TXD_2" O R 4300 4500 50
+F23 "ATM_SCK_1" O R 4300 4700 50
+F24 "ATM_SDA_1" B R 4300 3250 50
+F25 "ATM_SCL_1" O R 4300 3350 50
+F26 "ATM_PA3" T R 4300 4350 50
+F27 "ATM_PB3" O R 4300 3850 50
+F28 "ATM_PB4" O R 4300 3950 50
 $EndSheet
 $Comp
@@
 F8 "XBEE_SLEEP" I R 2400 4650 50
 F9 "XBEE_RESET" I R 2400 4750 50
-F10 "XBEE_ENABLE" I R 2400 4850 50
-F11 "XBEE_AD1" B R 2400 5650 50
-F12 "XBEE_VREF" U R 2400 5750 50
-F13 "XBEE_PWM0" B R 2400 5850 50
-F14 "XBEE_PWM1" B R 2400 5950 50
-F15 "XBEE_D18" B R 2400 6050 50
-F16 "RF_IRQ" O R 2400 5050 50
-F17 "RF_CE" I R 2400 4950 50
+F10 "XBEE_AD1" B R 2400 5650 50
+F11 "XBEE_VREF" U R 2400 5750 50
+F12 "XBEE_PWM0" B R 2400 5850 50
+F13 "XBEE_PWM1" B R 2400 5950 50
+F14 "XBEE_D18" B R 2400 6050 50
+F15 "RF_IRQ" O R 2400 5050 50
+F16 "RF_CE" I R 2400 4950 50
 $EndSheet
 Wire Wire Line
@@
 	2400 3250 2900 3250
 Wire Wire Line
-	2400 2500 2900 2500
-Wire Wire Line
-	2400 2600 2900 2600
-Wire Wire Line
-	2400 2700 2900 2700
-Wire Wire Line
 	2400 3650 2900 3650
 Wire Wire Line
 	2900 3750 2400 3750
-Wire Wire Line
-	2400 4850 2900 4850
 Wire Wire Line
 	2400 5050 2900 5050
@@
 Wire Wire Line
 	4300 3950 4800 3950
+$Sheet
+S 1000 2250 1400 1100
+U 5F86FCBB
+F0 "Sensors" 50
+F1 "SmartSensor_Sensors.sch" 50
+F2 "SDA" B R 2400 2900 50
+F3 "SCL" I R 2400 3000 50
+F4 "RESET" I R 2400 2350 50
+F5 "CO2_INT" O R 2400 3150 50
+F6 "CO2_WAKE" O R 2400 3250 50
+$EndSheet
 $EndSCHEMATC
