File: Hardware/SmartSensor_Communication.sch (KiCad schematic (older format))
At the start: 12 parts, among them IC3 XB24CZ7PIT-004, J7 Conn_01x02_Male, J8 Conn_01x06_Male, J9 Conn_02x04_Odd_Even, Q5 DMG2301L

Commit message: Added final version 1.2 to the repository
Parts:
- removed Q5: DMG2301L, Package_TO_SOT_SMD:SOT-23, symbol Transistor_FET:DMG2301L
- removed R11: 100k, Resistor_SMD:R_0805_2012Metric, symbol Device:R_Small
Connections:
- net +3V3: now also C15.1, C16.1, C17.1, IC3.1 (VCC), J9.7 (Pin_7)
- no-connect marks 4 -> 5
Changed lines of the file:
@@
 $Descr A4 11693 8268
 encoding utf-8
-Sheet 5 6
+Sheet 4 6
 Title "SmartSensor"
-Date "2021-03-19"
-Rev "1.1"
+Date "2021-06-14"
+Rev "1.2"
 Comp "Avans Hogeschool"
 Comment1 "Maurice Snoeren"
@@
 	1    0    0    -1
 $EndComp
-Wire Wire Line
-	3800 2150 3750 2150
-Text GLabel 3750 2150 0    50   Input ~ 0
-XBEE_ENABLE
-Wire Wire Line
-	3800 2100 3800 2150
-Wire Wire Line
-	3800 1900 4100 1900
-$Comp
-L Device:R_Small R11
-U 1 1 60078572
-P 3800 2000
-F 0 "R11" H 3650 1950 50  0000 L CNN
-F 1 "100k" V 3900 1900 50  0000 L CNN
-F 2 "Resistor_SMD:R_0805_2012Metric" H 3800 2000 50  0001 C CNN
-F 3 "~" H 3800 2000 50  0001 C CNN
-	1    3800 2000
-	-1   0    0    1
-$EndComp
-Connection ~ 3800 2150
-$Comp
-L Transistor_FET:DMG2301L Q5
-U 1 1 6007857A
-P 4000 2150
-F 0 "Q5" H 4204 2196 50  0000 L CNN
-F 1 "DMG2301L" H 4204 2105 50  0000 L CNN
-F 2 "Package_TO_SOT_SMD:SOT-23" H 4200 2075 50  0001 L CIN
-F 3 "https://www.diodes.com/assets/Datasheets/DMG2301L.pdf" H 4000 2150 50  0001 L CNN
-	1    4000 2150
-	1    0    0    1
-$EndComp
 $Comp
 L power:+3.3V #PWR032
 U 1 1 60078580
-P 4100 1900
-F 0 "#PWR032" H 4100 1750 50  0001 C CNN
-F 1 "+3.3V" H 4115 2073 50  0000 C CNN
-F 2 "" H 4100 1900 50  0001 C CNN
-F 3 "" H 4100 1900 50  0001 C CNN
-	1    4100 1900
-	1    0    0    -1
-$EndComp
-Connection ~ 4100 1900
-Wire Wire Line
-	4100 1950 4100 1900
+P 4100 2150
+F 0 "#PWR032" H 4100 2000 50  0001 C CNN
+F 1 "+3.3V" H 4115 2323 50  0000 C CNN
+F 2 "" H 4100 2150 50  0001 C CNN
+F 3 "" H 4100 2150 50  0001 C CNN
+	1    4100 2150
+	1    0    0    -1
+$EndComp
 Wire Wire Line
 	4100 2350 4100 2900
@@
 Text GLabel 1600 6600 2    50   Input ~ 0
 XBEE_PWM1
-Text GLabel 1600 6100 2    50   Input ~ 0
-XBEE_RF_ENABLE
 Text GLabel 4000 5250 2    50   Input ~ 0
 XBEE_UART_RTS
@@
 Text HLabel 1500 6000 0    50   Input ~ 0
 XBEE_RESET
-Text HLabel 1500 6100 0    50   Input ~ 0
-XBEE_ENABLE
 Text HLabel 1500 6300 0    50   BiDi ~ 0
 XBEE_AD1
@@
 Wire Wire Line
 	1600 6000 1500 6000
-Wire Wire Line
-	1500 6100 1600 6100
 Wire Wire Line
 	1600 6300 1500 6300
@@
 Text Notes 8300 3200 0    50   ~ 0
 SWITCH COMMISSION
+Wire Wire Line
+	4100 2150 4100 2350
+NoConn ~ 7800 -150
 $EndSCHEMATC
