File: Hardware/SmartSensor_MainController.sch (KiCad schematic (older format))
At the start: 26 parts, among them IC4 ATECC608B-SSHDA-B, J4 Conn_01x06_Male, J5 Conn_02x05_Odd_Even, J6 Conn_02x05_Odd_Even, U3 MCP7940N-xSN, U4 ATmega324PB-AU, Y1 20MHz, Y2 Crystal

Commit message: Added final version 1.2 to the repository
Parts:
- added D6: GREEN, LED_SMD:LED_0805_2012Metric, symbol Device:LED_Small
- added R4: 210, Resistor_SMD:R_0805_2012Metric, symbol Device:R_Small
- added R5: 100k, Resistor_SMD:R_0805_2012Metric, symbol Device:R_Small
Connections:
- net +3V3: now also R4.2, R5.1
- net RTC_MFP: now also R5.2
- net CO2_ENABLE renamed LED_2
- net LED_2: now also D6.1 (K)
- net LS_ENABLE: no longer names the net of U4.25 (PC6)
- net THS_ENABLE: no longer names the net of U4.26 (PC7)
- net XBEE_ENABLE: no longer names the net of U4.32 (PA5)
- new net: D6.2 (A), R4.1
- no-connect marks 11 -> 16
Other:
- moved on the sheet: D3, R9
Changed lines of the file:
@@
 $Descr A4 11693 8268
 encoding utf-8
-Sheet 4 6
+Sheet 3 6
 Title "SmartSensor"
-Date "2021-03-20"
-Rev "1.1"
+Date "2021-06-14"
+Rev "1.2"
 Comp "Avans Hogeschool"
 Comment1 "Maurice Snoeren"
@@
 Wire Wire Line
 	3900 6200 3900 6500
-Text GLabel 2100 5900 0    50   Input ~ 0
+Text GLabel 2000 5900 0    50   Input ~ 0
 SCL_MAIN
-Text GLabel 2100 6000 0    50   Input ~ 0
+Text GLabel 2000 6000 0    50   Input ~ 0
 SDA_MAIN
-Wire Wire Line
-	2100 5900 2150 5900
-Wire Wire Line
-	2100 6000 2150 6000
-Wire Wire Line
-	2100 6200 2150 6200
-Text GLabel 2100 6200 0    50   Input ~ 0
+Text GLabel 2000 6200 0    50   Input ~ 0
 RTC_MFP
 $Comp
 L Device:R_Small R?
 U 1 1 5F85783F
-P 5700 2850
+P 5700 2700
 AR Path="/5F85783F" Ref="R?"  Part="1"
 AR Path="/5F76931A/5F85783F" Ref="R9"  Part="1"
-F 0 "R9" V 5650 2600 50  0000 L CNN
-F 1 "210" V 5600 2800 50  0000 L CNN
-F 2 "Resistor_SMD:R_0805_2012Metric" H 5700 2850 50  0001 C CNN
-F 3 "~" H 5700 2850 50  0001 C CNN
-	1    5700 2850
+F 0 "R9" V 5650 2450 50  0000 L CNN
+F 1 "210" V 5600 2650 50  0000 L CNN
+F 2 "Resistor_SMD:R_0805_2012Metric" H 5700 2700 50  0001 C CNN
+F 3 "~" H 5700 2700 50  0001 C CNN
+	1    5700 2700
 	0    1    1    0
 $EndComp
@@
 L Device:LED_Small D?
 U 1 1 5F857845
-P 5950 2850
+P 5950 2700
 AR Path="/5F857845" Ref="D?"  Part="1"
 AR Path="/5F76931A/5F857845" Ref="D3"  Part="1"
-F 0 "D3" H 6000 2750 50  0000 C CNN
-F 1 "RED" H 5800 2750 50  0000 C CNN
-F 2 "LED_SMD:LED_0805_2012Metric" V 5950 2850 50  0001 C CNN
-F 3 "~" V 5950 2850 50  0001 C CNN
-	1    5950 2850
+F 0 "D3" H 6000 2600 50  0000 C CNN
+F 1 "RED" H 5800 2600 50  0000 C CNN
+F 2 "LED_SMD:LED_0805_2012Metric" V 5950 2700 50  0001 C CNN
+F 3 "~" V 5950 2700 50  0001 C CNN
+	1    5950 2700
 	-1   0    0    1
 $EndComp
@@
 L power:+3.3V #PWR?
 U 1 1 5F85784B
-P 5400 2750
+P 5400 2600
 AR Path="/5F85784B" Ref="#PWR?"  Part="1"
 AR Path="/5F76931A/5F85784B" Ref="#PWR020"  Part="1"
-F 0 "#PWR020" H 5400 2600 50  0001 C CNN
-F 1 "+3.3V" H 5415 2923 50  0000 C CNN
-F 2 "" H 5400 2750 50  0001 C CNN
-F 3 "" H 5400 2750 50  0001 C CNN
-	1    5400 2750
-	1    0    0    -1
-$EndComp
-Text GLabel 6100 2850 2    50   Input ~ 0
+F 0 "#PWR020" H 5400 2450 50  0001 C CNN
+F 1 "+3.3V" H 5415 2773 50  0000 C CNN
+F 2 "" H 5400 2600 50  0001 C CNN
+F 3 "" H 5400 2600 50  0001 C CNN
+	1    5400 2600
+	1    0    0    -1
+$EndComp
+Text GLabel 6100 2700 2    50   Input ~ 0
 LED_1
 Wire Wire Line
-	6050 2850 6100 2850
-Wire Wire Line
-	5400 2750 5400 2850
-Wire Wire Line
-	5600 2850 5400 2850
-Wire Wire Line
-	5850 2850 5800 2850
+	6050 2700 6100 2700
+Wire Wire Line
+	5400 2600 5400 2700
+Wire Wire Line
+	5600 2700 5400 2700
+Wire Wire Line
+	5850 2700 5800 2700
 $Comp
 L Connector_Generic:Conn_02x05_Odd_Even J?
@@
 RF_IRQ
 Wire Wire Line
-	4000 2200 3950 2200
-Wire Wire Line
 	4000 2300 3950 2300
 Wire Wire Line
 	4000 2400 3950 2400
 Wire Wire Line
-	3950 4200 4000 4200
-Wire Wire Line
-	4000 4100 3950 4100
-Wire Wire Line
 	2750 4100 2700 4100
-Wire Wire Line
-	2750 4000 2700 4000
 Text HLabel 3950 3000 2    50   Output ~ 0
 ATM_PB4
@@
 Wire Wire Line
 	3950 2600 4000 2600
-Text HLabel 4000 2200 2    50   Output ~ 0
-XBEE_ENABLE
 Text HLabel 4000 2700 2    50   Output ~ 0
 XBEE_SLEEP
@@
 Text HLabel 4000 2400 2    50   Output ~ 0
 CO2_INT
-Text HLabel 4000 4200 2    50   Output ~ 0
-THS_ENABLE
-Text HLabel 4000 4100 2    50   Output ~ 0
-LS_ENABLE
-Text HLabel 2700 4000 0    50   Output ~ 0
-CO2_ENABLE
 Wire Wire Line
 	2700 1700 2750 1700
@@
 Text Notes 5450 3700 0    50   ~ 0
 SWITCH GENERAL
+Text GLabel 2700 4000 0    50   Input ~ 0
+LED_2
+Wire Wire Line
+	2700 4000 2750 4000
+$Comp
+L Device:R_Small R?
+U 1 1 60C57333
+P 5700 2900
+AR Path="/60C57333" Ref="R?"  Part="1"
+AR Path="/5F76931A/60C57333" Ref="R4"  Part="1"
+F 0 "R4" V 5650 2650 50  0000 L CNN
+F 1 "210" V 5600 2850 50  0000 L CNN
+F 2 "Resistor_SMD:R_0805_2012Metric" H 5700 2900 50  0001 C CNN
+F 3 "~" H 5700 2900 50  0001 C CNN
+	1    5700 2900
+	0    1    1    0
+$EndComp
+$Comp
+L Device:LED_Small D?
+U 1 1 60C57339
+P 5950 2900
+AR Path="/60C57339" Ref="D?"  Part="1"
+AR Path="/5F76931A/60C57339" Ref="D6"  Part="1"
+F 0 "D6" H 6000 2800 50  0000 C CNN
+F 1 "GREEN" H 5800 2800 50  0000 C CNN
+F 2 "LED_SMD:LED_0805_2012Metric" V 5950 2900 50  0001 C CNN
+F 3 "~" V 5950 2900 50  0001 C CNN
+	1    5950 2900
+	-1   0    0    1
+$EndComp
+Text GLabel 6100 2900 2    50   Input ~ 0
+LED_2
+Wire Wire Line
+	6050 2900 6100 2900
+Wire Wire Line
+	5600 2900 5400 2900
+Wire Wire Line
+	5850 2900 5800 2900
+Wire Wire Line
+	5400 2700 5400 2900
+Connection ~ 5400 2700
+$Comp
+L Device:R_Small R?
+U 1 1 60C733DE
+P 2100 5550
+AR Path="/60C733DE" Ref="R?"  Part="1"
+AR Path="/5F76931A/60C733DE" Ref="R5"  Part="1"
+F 0 "R5" H 2159 5596 50  0000 L CNN
+F 1 "100k" V 2000 5500 50  0000 L CNN
+F 2 "Resistor_SMD:R_0805_2012Metric" H 2100 5550 50  0001 C CNN
+F 3 "~" H 2100 5550 50  0001 C CNN
+	1    2100 5550
+	1    0    0    -1
+$EndComp
+Wire Wire Line
+	2000 5900 2150 5900
+Wire Wire Line
+	2000 6000 2150 6000
+Wire Wire Line
+	2000 6200 2100 6200
+Wire Wire Line
+	2100 5650 2100 6200
+Connection ~ 2100 6200
+Wire Wire Line
+	2100 6200 2150 6200
+Wire Wire Line
+	2100 5450 2100 5350
+Wire Wire Line
+	2100 5350 2550 5350
+NoConn ~ 6350 3400
+NoConn ~ 6350 3500
+NoConn ~ 3950 4100
+NoConn ~ 3950 4200
+NoConn ~ 3950 2200
 $EndSCHEMATC
